Commit message: Wrote ddrive_rviz.launch.xml and got robot to show up in rviz

File: diff_drive/urdf/ddrive.urdf.xacro (robot description, xacro)
@@ -1,4 +1,4 @@
 <robot name="ddrive" xmlns:xacro="http://www.ros.org/wiki/xacro">
-    <xacro:property name="ddrive_yaml" value="$(find ddrive)/config/ddrive.yaml"/>
+    <xacro:property name="ddrive_yaml" value="$(find diff_drive)/config/ddrive.yaml"/>
     <xacro:property name="yaml_dict" value="${xacro.load_yaml(ddrive_yaml)['/**']['ros__parameters']}"/>
     <xacro:property name="base_length" value="${yaml_dict['base_length']}"/>
@@ -27,6 +27,5 @@
                 <box size="${base_length} ${base_width} ${base_height}"/>
             </geometry>
-            <material name="base"/>
-            <origin xyz="0 0 ${wheel_radius*2 + .05 + side_length/2}"/>
+            <material name="white"/>
         </visual>
         <collision>
@@ -141,5 +140,5 @@
         <parent link="bottom_caster_base"/>
         <child link="bottom_caster_wheel"/>
-        <origin rpy="{-pi/2} 0 0" xyz="0 0 ${-(.5*wheel_radius + .5*(wheel_radius - .5*base_height - 2*caster_wheel_radius))}"/>
+        <origin rpy="${-pi/2} 0 0" xyz="0 0 ${-(.5*wheel_radius + .5*(wheel_radius - .5*base_height - 2*caster_wheel_radius))}"/>
         <axis xyz= "0 0 1"/>
     </joint>
@@ -147,13 +146,6 @@
         <parent link="top_caster_base"/>
         <child link="top_caster_wheel"/>
-        <origin rpy="{-pi/2} 0 0" xyz="0 0 ${-(.5*wheel_radius + .5*(wheel_radius - .5*base_height - 2*caster_wheel_radius))}"/>
+        <origin rpy="${-pi/2} 0 0" xyz="0 0 ${-(.5*wheel_radius + .5*(wheel_radius - .5*base_height - 2*caster_wheel_radius))}"/>
         <axis xyz= "0 0 1"/>
     </joint>
-    <joint name="connector_to_platform" type="revolute">
-        <parent link="base_platform_connector"/>
-        <child link="platform"/>
-        <origin xyz="0 0 ${(platform_height - .05 - (wheel_radius*2 + .05 + side_length))/2}"/>
-        <limit effort="1000.0" lower="${-pi/4}" upper="${pi/4}" velocity="0.5"/>
-        <axis xyz="1 0 0"/>
-    </joint>
 </robot>

Commit message: Got robot to show up properly in rviz

File: diff_drive/urdf/ddrive.urdf.xacro (robot description, xacro)
@@ -116,5 +116,5 @@
         <parent link="base_link"/>
         <child link="left_wheel"/>
-        <origin rpy="${-pi/2} 0 0" xyz="${center_to_wheel} ${.5*base_width} 0"/>
+        <origin rpy="${-pi/2} 0 0" xyz="${center_to_wheel} ${.5*(base_width + wheel_thickness)} 0"/>
         <axis xyz= "0 0 1"/>
     </joint>
@@ -122,5 +122,5 @@
         <parent link="base_link"/>
         <child link="right_wheel"/>
-        <origin rpy="${-pi/2} 0 0" xyz="${center_to_wheel} ${-.5*base_width} 0"/>
+        <origin rpy="${-pi/2} 0 0" xyz="${center_to_wheel} ${-.5*(base_width + wheel_thickness)} 0"/>
         <axis xyz= "0 0 1"/>
     </joint>
@@ -128,5 +128,5 @@
         <parent link="base_link"/>
         <child link="bottom_caster_base"/>
-        <origin xyz="${center_to_wheel} 0 ${-(.5*base_height + .5*(wheel_radius - .5*base_height - 2*caster_wheel_radius))}"/>
+        <origin xyz="${-center_to_wheel} 0 ${-((wheel_radius - .5*base_height - 2*caster_wheel_radius)/2 + base_height/2)}"/>
         <axis xyz= "0 0 1"/>
     </joint>
@@ -134,5 +134,5 @@
         <parent link="base_link"/>
         <child link="top_caster_base"/>
-        <origin rpy="${pi} 0 0" xyz="${center_to_wheel} 0 ${.5*base_height + .5*(wheel_radius - .5*base_height - 2*caster_wheel_radius)}"/>
+        <origin rpy="${pi} 0 0" xyz="${-center_to_wheel} 0 ${((wheel_radius - .5*base_height - 2*caster_wheel_radius)/2 + base_height/2)}"/>
         <axis xyz= "0 0 1"/>
     </joint>
@@ -140,5 +140,5 @@
         <parent link="bottom_caster_base"/>
         <child link="bottom_caster_wheel"/>
-        <origin rpy="${-pi/2} 0 0" xyz="0 0 ${-(.5*wheel_radius + .5*(wheel_radius - .5*base_height - 2*caster_wheel_radius))}"/>
+        <origin rpy="${-pi/2} 0 0" xyz="0 0 ${-((wheel_radius - .5*base_height - 2*caster_wheel_radius)/2 + caster_wheel_radius/2)}"/>
         <axis xyz= "0 0 1"/>
     </joint>
@@ -146,5 +146,5 @@
         <parent link="top_caster_base"/>
         <child link="top_caster_wheel"/>
-        <origin rpy="${-pi/2} 0 0" xyz="0 0 ${-(.5*wheel_radius + .5*(wheel_radius - .5*base_height - 2*caster_wheel_radius))}"/>
+        <origin rpy="${-pi/2} 0 0" xyz="0 0 ${-((wheel_radius - .5*base_height - 2*caster_wheel_radius)/2 + caster_wheel_radius/2)}"/>
         <axis xyz= "0 0 1"/>
     </joint>

Commit message: Made edit to ddrive.urdf.xacro

File: diff_drive/urdf/ddrive.urdf.xacro (robot description, xacro)
@@ -7,6 +7,5 @@
     <xacro:property name="wheel_radius" value="${yaml_dict['wheel_radius']}"/>
     <xacro:property name="wheel_thickness" value="${yaml_dict['wheel_thickness']}"/>
-    <xacro:property name="caster_base_radius" value="${yaml_dict['caster_base_radius']}"/>
-    <xacro:property name="caster_wheel_radius" value="${yaml_dict['caster_wheel_radius']}"/>
+    <xacro:property name="caster_radius" value="${yaml_dict['caster_radius']}"/>
     <xacro:property name="center_to_wheel" value="${yaml_dict['center_to_wheel']}"/>
     <material name="blue">
@@ -61,21 +60,8 @@
         </collision>
     </link>
-    <link name="bottom_caster_wheel">
+    <link name="bottom_caster">
         <visual>
             <geometry>
-                <cylinder length="${2*caster_base_radius}" radius="${caster_wheel_radius}"/>
-            </geometry>
-            <material name="black"/>
-        </visual>
-        <collision>
-            <geometry>
-                <cylinder length="${2*caster_base_radius}" radius="${caster_wheel_radius}"/>
-            </geometry>
-        </collision>
-    </link>
-    <link name="bottom_caster_base">
-        <visual>
-            <geometry>
-                <cylinder length="${wheel_radius - .5*base_height - 2*caster_wheel_radius}" radius="${caster_base_radius}"/>
+                <sphere radius="${caster_radius}"/>
             </geometry>
             <material name="red"/>
@@ -83,25 +69,12 @@
         <collision>
             <geometry>
-                <cylinder length="${wheel_radius - .5*base_height - 2*caster_wheel_radius}" radius="${caster_base_radius}"/>
+                <sphere radius="${caster_radius}"/>
             </geometry>
         </collision>
     </link>
-    <link name="top_caster_wheel">
+    <link name="top_caster">
         <visual>
             <geometry>
-                <cylinder length="${2*caster_base_radius}" radius="${caster_wheel_radius}"/>
-            </geometry>
-            <material name="black"/>
-        </visual>
-        <collision>
-            <geometry>
-                <cylinder length="${2*caster_base_radius}" radius="${caster_wheel_radius}"/>
-            </geometry>
-        </collision>
-    </link>
-    <link name="top_caster_base">
-        <visual>
-            <geometry>
-                <cylinder length="${wheel_radius - .5*base_height - 2*caster_wheel_radius}" radius="${caster_base_radius}"/>
+                <sphere radius="${caster_radius}"/>
             </geometry>
             <material name="blue"/>
@@ -109,5 +82,5 @@
         <collision>
             <geometry>
-                <cylinder length="${wheel_radius - .5*base_height - 2*caster_wheel_radius}" radius="${caster_base_radius}"/>
+                <sphere radius="${caster_radius}"/>
             </geometry>
         </collision>
@@ -125,26 +98,14 @@
         <axis xyz= "0 0 1"/>
     </joint>
-    <joint name="base_to_bottom_caster" type="continuous">
+    <joint name="base_to_bottom_caster" type="fixed">
         <parent link="base_link"/>
-        <child link="bottom_caster_base"/>
-        <origin xyz="${-center_to_wheel} 0 ${-((wheel_radius - .5*base_height - 2*caster_wheel_radius)/2 + base_height/2)}"/>
+        <child link="bottom_caster"/>
+        <origin xyz="${-center_to_wheel} 0 ${-(base_height/2 + caster_radius)}"/>
         <axis xyz= "0 0 1"/>
     </joint>
-    <joint name="base_to_top_caster" type="continuous">
+    <joint name="base_to_top_caster" type="fixed">
         <parent link="base_link"/>
-        <child link="top_caster_base"/>
-        <origin rpy="${pi} 0 0" xyz="${-center_to_wheel} 0 ${((wheel_radius - .5*base_height - 2*caster_wheel_radius)/2 + base_height/2)}"/>
-        <axis xyz= "0 0 1"/>
-    </joint>
-    <joint name="bottom_caster_to_wheel" type="continuous">
-        <parent link="bottom_caster_base"/>
-        <child link="bottom_caster_wheel"/>
-        <origin rpy="${-pi/2} 0 0" xyz="0 0 ${-((wheel_radius - .5*base_height - 2*caster_wheel_radius)/2 + caster_wheel_radius/2)}"/>
-        <axis xyz= "0 0 1"/>
-    </joint>
-    <joint name="top_caster_to_wheel" type="continuous">
-        <parent link="top_caster_base"/>
-        <child link="top_caster_wheel"/>
-        <origin rpy="${-pi/2} 0 0" xyz="0 0 ${-((wheel_radius - .5*base_height - 2*caster_wheel_radius)/2 + caster_wheel_radius/2)}"/>
+        <child link="top_caster"/>
+        <origin xyz="${-center_to_wheel} 0 ${base_height/2 + caster_radius}"/>
         <axis xyz= "0 0 1"/>
     </joint>

Commit message: Added inertial tags for ddrive.urdf.xacro

File: diff_drive/urdf/ddrive.urdf.xacro (robot description, xacro)
@@ -33,4 +33,15 @@
             </geometry>
         </collision>
+        <inertial>
+            <mass value="2" />
+            <inertia
+                ixx="0.181"
+                ixy="0"
+                ixz="0"
+                iyy="0.681"
+                iyz="0"
+                izz="0.833"
+            />
+        </inertial>
     </link>
     <link name="left_wheel">
@@ -46,4 +57,15 @@
             </geometry>
         </collision>
+        <inertial>
+            <mass value="1"/>
+            <inertia
+                ixx="0.064375"
+                ixy="0"
+                ixz="0"
+                iyy="0.064375"
+                iyz="0"
+                izz="0.125"
+            />
+        </inertial>
     </link>
     <link name="right_wheel">
@@ -59,4 +81,15 @@
             </geometry>
         </collision>
+        <inertial>
+            <mass value="1"/>
+            <inertia
+                ixx="0.064375"
+                ixy="0"
+                ixz="0"
+                iyy="0.064375"
+                iyz="0"
+                izz="0.125"
+            />
+        </inertial>
     </link>
     <link name="bottom_caster">
@@ -72,4 +105,15 @@
             </geometry>
         </collision>
+        <inertial>
+            <mass value="1"/>
+            <inertia
+                ixx="0.01225"
+                ixy="0"
+                ixz="0"
+                iyy="0.01225"
+                iyz="0"
+                izz="0.01225"
+            />
+        </inertial>
     </link>
     <link name="top_caster">
@@ -85,4 +129,15 @@
             </geometry>
         </collision>
+        <inertial>
+            <mass value="1"/>
+            <inertia
+                ixx="0.01225"
+                ixy="0"
+                ixz="0"
+                iyy="0.01225"
+                iyz="0"
+                izz="0.01225"
+            />
+        </inertial>
     </link>
     <joint name="base_to_left_wheel" type="continuous">

Commit message: flip.py moves the robot, but does not move it correctly

File: diff_drive/urdf/ddrive.urdf.xacro (robot description, xacro)
@@ -34,12 +34,12 @@
         </collision>
         <inertial>
-            <mass value="2" />
+            <mass value="1" />
             <inertia
-                ixx="0.181"
+                ixx="0.09"
                 ixy="0"
                 ixz="0"
-                iyy="0.681"
+                iyy="0.09"
                 iyz="0"
-                izz="0.833"
+                izz="0.166"
             />
         </inertial>
@@ -104,4 +104,5 @@
                 <sphere radius="${caster_radius}"/>
             </geometry>
+            <contact_coefficients mu="0.0"/>
         </collision>
         <inertial>
@@ -128,4 +129,5 @@
                 <sphere radius="${caster_radius}"/>
             </geometry>
+            <contact_coefficients mu="0.0"/>
         </collision>
         <inertial>
