Commit message: Got robot to show up in gazebo and modified ddrive.launch.xml

File: diff_drive/urdf/ddrive.gazebo.xacro (robot description, xacro)
@@ -16,5 +16,5 @@
             <left_joint>base_to_left_wheel</left_joint>
             <right_joint>base_to_right_wheel</right_joint>
-            <wheel_separation>1.25</wheel_separation>
+            <wheel_separation>1.15</wheel_separation>
             <wheel_radius>.5</wheel_radius>
             <odom_publish_frequency>50</odom_publish_frequency>

File: diff_drive/urdf/ddrive.urdf.xacro (robot description, xacro)
@@ -18,6 +18,6 @@
         <color rgba="1 1 1 1"/>
     </material>
-    <material name="black">
-        <color rgba="0 0 0 1"/>
+    <material name="green">
+        <color rgba="0 0.8 0 1"/>
     </material>
     <link name="base_link">
@@ -50,5 +50,5 @@
                 <cylinder length="${wheel_thickness}" radius="${wheel_radius}"/>
             </geometry>
-            <material name="black"/>
+            <material name="green"/>
         </visual>
         <collision>
@@ -74,5 +74,5 @@
                 <cylinder length="${wheel_thickness}" radius="${wheel_radius}"/>
             </geometry>
-            <material name="black"/>
+            <material name="green"/>
         </visual>
         <collision>

Commit message: Made changes to inertia properties and removed friction; fixed flip node

File: diff_drive/urdf/ddrive.gazebo.xacro (robot description, xacro)
@@ -10,4 +10,12 @@
     <xacro:property name="caster_radius" value="${yaml_dict['caster_radius']}"/>
     <xacro:property name="center_to_wheel" value="${yaml_dict['center_to_wheel']}"/>
+    <gazebo reference="top_caster">
+        <mu1>0.0</mu1>
+        <mu2>0.0</mu2>
+    </gazebo>
+    <gazebo reference="bottom_caster">
+        <mu1>0.0</mu1>
+        <mu2>0.0</mu2>
+    </gazebo>
     <gazebo>
         <plugin
@@ -22,8 +30,8 @@
             <child_frame_id>base_link</child_frame_id>
         </plugin>
-      <plugin
-          filename="libgz-sim-joint-state-publisher-system.so"
-          name="gz::sim::systems::JointStatePublisher">
-          </plugin>
+        <plugin
+            filename="libgz-sim-joint-state-publisher-system.so"
+            name="gz::sim::systems::JointStatePublisher">
+        </plugin>
      </gazebo>
 </robot>

File: diff_drive/urdf/ddrive.urdf.xacro (robot description, xacro)
@@ -9,4 +9,13 @@
     <xacro:property name="caster_radius" value="${yaml_dict['caster_radius']}"/>
     <xacro:property name="center_to_wheel" value="${yaml_dict['center_to_wheel']}"/>
+    <xacro:property name="base_mass" value=".05"/>
+    <xacro:property name="wheel_mass" value="5"/>
+    <xacro:property name="caster_mass" value="0.001"/>
+    <xacro:property name="base_ixx" value="${base_mass*(base_width**2 + base_height**2)/12}"/>
+    <xacro:property name="base_iyy" value="${base_mass*(base_length**2 + base_height**2)/12}"/>
+    <xacro:property name="base_izz" value="${base_mass*(base_width**2 + base_length**2)/12}"/>
+    <xacro:property name="wheel_ixx" value="${wheel_mass*(3*(wheel_radius**2) + wheel_thickness**2)/12}"/>
+    <xacro:property name="wheel_izz" value="${wheel_mass*(wheel_radius**2)/2}"/>
+    <xacro:property name="caster_ixx" value="${caster_mass*2*(caster_radius**2)/5}"/>
     <material name="blue">
         <color rgba="0 0 0.8 1"/>
@@ -36,10 +45,10 @@
             <mass value="1" />
             <inertia
-                ixx="0.09"
+                ixx="${base_ixx}"
                 ixy="0"
                 ixz="0"
-                iyy="0.09"
+                iyy="${base_iyy}"
                 iyz="0"
-                izz="0.166"
+                izz="${base_izz}"
             />
         </inertial>
@@ -60,10 +69,10 @@
             <mass value="1"/>
             <inertia
-                ixx="0.064375"
+                ixx="${wheel_ixx}"
                 ixy="0"
                 ixz="0"
-                iyy="0.064375"
+                iyy="${wheel_ixx}"
                 iyz="0"
-                izz="0.125"
+                izz="${wheel_izz}"
             />
         </inertial>
@@ -84,10 +93,10 @@
             <mass value="1"/>
             <inertia
-                ixx="0.064375"
+                ixx="${wheel_ixx}"
                 ixy="0"
                 ixz="0"
-                iyy="0.064375"
+                iyy="${wheel_ixx}"
                 iyz="0"
-                izz="0.125"
+                izz="${wheel_izz}"
             />
         </inertial>
@@ -109,10 +118,10 @@
             <mass value="1"/>
             <inertia
-                ixx="0.01225"
+                ixx="${caster_ixx}"
                 ixy="0"
                 ixz="0"
-                iyy="0.01225"
+                iyy="${caster_ixx}"
                 iyz="0"
-                izz="0.01225"
+                izz="${caster_ixx}"
             />
         </inertial>
@@ -134,10 +143,10 @@
             <mass value="1"/>
             <inertia
-                ixx="0.01225"
+                ixx="${caster_ixx}"
                 ixy="0"
                 ixz="0"
-                iyy="0.01225"
+                iyy="${caster_ixx}"
                 iyz="0"
-                izz="0.01225"
+                izz="${caster_ixx}"
             />
         </inertial>

Commit message: Made edits to doctstrings in flip node; removed unnecessary xacro properties in ddrive.gazebo.xacro file; cited sources; updated README

File: diff_drive/urdf/ddrive.gazebo.xacro (robot description, xacro)
@@ -3,11 +3,7 @@
     <xacro:property name="ddrive_yaml" value="$(find diff_drive)/config/ddrive.yaml"/>
     <xacro:property name="yaml_dict" value="${xacro.load_yaml(ddrive_yaml)['/**']['ros__parameters']}"/>
-    <xacro:property name="base_length" value="${yaml_dict['base_length']}"/>
     <xacro:property name="base_width" value="${yaml_dict['base_width']}"/>
-    <xacro:property name="base_height" value="${yaml_dict['base_height']}"/>
     <xacro:property name="wheel_radius" value="${yaml_dict['wheel_radius']}"/>
     <xacro:property name="wheel_thickness" value="${yaml_dict['wheel_thickness']}"/>
-    <xacro:property name="caster_radius" value="${yaml_dict['caster_radius']}"/>
-    <xacro:property name="center_to_wheel" value="${yaml_dict['center_to_wheel']}"/>
     <gazebo reference="top_caster">
         <mu1>0.0</mu1>
